File: _autosave-_autosave-24S_Counter.kicad_pcb (KiCad board)
At the start: 2 copper layers, 84 x 74.5 mm, 32 parts, among them J1 +5V, J2 EXT_CLK, SW1 EN, SW2 RST, U1 74LS192, U2 74LS192, U3 74LS48, U4 74LS48, U5 SM420561N, U6 SM420561N

Commit message: done
Routing:
- net /CLK: track 9.86 -> 24.8 mm, vias 0 -> 1
- net /+5V: track 131.6 -> 144.2 mm
Other:
- board text added: "24 SECOND COUNTER Design Engineer: Chrischele Palacios Date: 13 April 2026"
Changed lines of the file:
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@@
 		)
 		(embedded_fonts no)
+		(model "${KIPRJMOD}/my_lib/my_3D/74LS48.step"
+			(offset
+				(xyz 0 0 0)
+			)
+			(scale
+				(xyz 1 1 1)
+			)
+			(rotate
+				(xyz -90 -0 -0)
+			)
+		)
 	)
 	(footprint "Resistor_SMD:R_1206_3216Metric_Pad1.30x1.75mm_HandSolder"
@@
 		)
 		(embedded_fonts no)
+		(model "${KIPRJMOD}/my_lib/my_3D/74LS48.step"
+			(offset
+				(xyz 0 0 0)
+			)
+			(scale
+				(xyz 1 1 1)
+			)
+			(rotate
+				(xyz -90 -0 -0)
+			)
+		)
 	)
 	(footprint "Resistor_SMD:R_1206_3216Metric_Pad1.30x1.75mm_HandSolder"
@@
 		(tags "resistor handsolder")
 		(property "Reference" "R16"
-			(at 0 -1.83 0)
+			(at 0 0 0)
 			(layer "F.SilkS")
 			(effects
@@
 		)
 		(embedded_fonts no)
+		(model "${KIPRJMOD}/my_lib/my_3D/tact_switch.step"
+			(offset
+				(xyz 0 0 0)
+			)
+			(scale
+				(xyz 1 1 1)
+			)
+			(rotate
+				(xyz -90 -0 -0)
+			)
+		)
 	)
 	(footprint "my_footprints:slide_switch_2.54mm"
@@
 		(at 102 75 90)
 		(property "Reference" "SW1"
-			(at -2.54 -3.175 90)
+			(at -3.5 -1 90)
 			(layer "F.SilkS")
 			(effects
@@
 		)
 		(embedded_fonts no)
+		(model "${KIPRJMOD}/my_lib/my_3D/slide_switch.step"
+			(offset
+				(xyz 0 0 0)
+			)
+			(scale
+				(xyz 1 1 1)
+			)
+			(rotate
+				(xyz 0 0 0)
+			)
+		)
 	)
 	(footprint "Display_7Segment:7SegmentLED_LTS6760_LTS6780"
@@
 		(tags "resistor handsolder")
 		(property "Reference" "R15"
-			(at 0 -1.83 0)
+			(at 0 0 0)
 			(layer "F.SilkS")
 			(effects
@@
 		(at 93.5 36.5 180)
 		(property "Reference" "J1"
-			(at -1.825 -8.635 0)
+			(at 0.5 -3.5 0)
 			(layer "F.SilkS")
 			(effects
@@
 		(layer "Edge.Cuts")
 	)
+	(gr_text "24 SECOND COUNTER\nDesign Engineer:\nChrischele Palacios\nDate:\n13 April 2026"
+		(at 102 34.5 0)
+		(layer "F.SilkS")
+		(effects
+			(font
+				(size 1.27 1.27)
+				(thickness 0.3175)
+				(bold yes)
+			)
+			(justify left bottom)
+		)
+	)
 	(segment
 		(start 139.31 69.61)
@@
 	)
 	(segment
+		(start 88.69 46.11)
+		(end 88.69 45.81)
+		(width 0.508)
+		(layer "B.Cu")
+		(net 1)
+	)
+	(segment
 		(start 106.58 46.3)
 		(end 109.12 46.3)
@@
 	)
 	(segment
+		(start 96 38.5)
+		(end 96 36.5)
+		(width 0.508)
+		(layer "B.Cu")
+		(net 1)
+	)
+	(segment
+		(start 88.69 45.81)
+		(end 96 38.5)
+		(width 0.508)
+		(layer "B.Cu")
+		(net 1)
+	)
+	(segment
 		(start 116.88 79.96)
 		(end 115.34 81.5)
@@
 	)
 	(segment
+		(start 113.08 77.42)
+		(end 113 77.5)
+		(width 0.2)
+		(layer "F.Cu")
+		(net 33)
+	)
+	(segment
 		(start 96 73)
 		(end 96 76.4)
@@
 	)
 	(segment
+		(start 116.88 77.42)
+		(end 113.08 77.42)
+		(width 0.2)
+		(layer "F.Cu")
+		(net 33)
+	)
+	(segment
 		(start 96 76.4)
 		(end 100.9 76.4)
@@
 		(net 33)
 	)
+	(via
+		(at 113 77.5)
+		(size 0.6)
+		(drill 0.3)
+		(layers "F.Cu" "B.Cu")
+		(net 33)
+	)
+	(segment
+		(start 102 77.5)
+		(end 104.5 77.5)
+		(width 0.381)
+		(layer "B.Cu")
+		(net 33)
+	)
+	(segment
+		(start 104.5 77.5)
+		(end 113 77.5)
+		(width 0.381)
+		(layer "B.Cu")
+		(net 33)
+	)
